Commit message: multi-robot localization 진행 중

File: follow_cart/urdf/convoy/jetbot.urdf (robot description, URDF)
Before this commit: robot JetBot, 6 links, 5 joints
Links:
- removed link left_wheel
- removed link lidar_link
- removed link right_wheel
- added link base_scan, mass 0.0; collision mesh filename=file://$(find follow_cart)/meshes/convoy/lidar-base.dae scale=1.0 1.0 1.0; visual mesh filename=file://$(find follow_cart)/meshes/convoy/lidar-base.dae scale=1.0 1.0 1.0
- added link imu_link
- added link wheel_left_link, mass 0.1; collision cylinder length=0.008 radius=0.030; visual mesh filename=file://$(find follow_cart)/meshes/convoy/JetBot-v3-Wheel.stl scale=0.001 0.001 0.001
- added link wheel_right_link, mass 0.1; collision cylinder length=0.008 radius=0.030; visual mesh filename=file://$(find follow_cart)/meshes/convoy/JetBot-v3-Wheel.stl scale=0.001 0.001 0.001
Joints:
- removed joint left_wheel_hinge
- removed joint right_wheel_hinge
- added joint imu_joint: type fixed, parent base_link, child imu_link, origin xyz=0 0 0.01
- added joint wheel_left_joint: type continuous, parent base_link, child wheel_left_link, origin xyz=0.03     0.05125  0.03 rpy=0       0       1.57079, axis 1  0  0
- added joint wheel_right_joint: type continuous, parent base_link, child wheel_right_link, origin xyz=0.03   -0.0595  0.03 rpy=0       0       1.57079, axis 1  0  0
- joint lidar_joint: child lidar_link -> base_scan

File: follow_cart/urdf/follow_cart/turtlebot3_waffle_pi.urdf (robot description, URDF)
Before this commit: robot turtlebot3_waffle_pi, 8 links, 7 joints
Links:
- removed link base_footprint
- removed link base_link
- removed link base_scan
- removed link caster_back_left_link
- removed link caster_back_right_link
- removed link imu_link
- removed link wheel_left_link
- removed link wheel_right_link
- added link fc1/base_footprint
- added link fc1/base_link, mass 1.3729096e+00; collision box size=0.266 0.266 0.094; visual mesh filename=file://$(find turtlebot3_description)/meshes/bases/waffle_p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 scale=0.001 0.001 0.001
- added link fc1/base_scan, mass 0.114; collision cylinder length=0.0315 radius=0.055; visual mesh filename=file://$(find turtlebot3_description)/meshes/sensors/lds.stl scale=0.001 0.001 0.001
- added link fc1/caster_back_left_link, mass 0.005; collision box size=0.030 0.009 0.020
- added link fc1/caster_back_right_link, mass 0.005; collision box size=0.030 0.009 0.020
- added link fc1/imu_link
- added link fc1/wheel_left_link, mass 2.8498940e-02; collision cylinder length=0.018 radius=0.033; visual mesh filename=file://$(find turtlebot3_description)/meshes/wheels/left_ti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 scale=0.001 0.001 0.001
- added link fc1/wheel_right_link, mass 2.8498940e-02; collision cylinder length=0.018 radius=0.033; visual mesh filename=file://$(find turtlebot3_description)/meshes/wheels/right_t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 scale=0.001 0.001 0.001
Joints:
- removed joint base_joint
- removed joint caster_back_left_joint
- removed joint caster_back_right_joint
- removed joint imu_joint
- removed joint scan_joint
- removed joint wheel_left_joint
- removed joint wheel_right_joint
- added joint fc1/base_joint: type fixed, parent fc1/base_footprint, child fc1/base_link, origin xyz=0 0 0.010 rpy=0 0 0
- added joint fc1/caster_back_left_joint: type fixed, parent fc1/base_link, child fc1/caster_back_left_link, origin xyz=-0.177 0.064 -0.004 rpy=-1.57 0 0
- added joint fc1/caster_back_right_joint: type fixed, parent fc1/base_link, child fc1/caster_back_right_link, origin xyz=-0.177 -0.064 -0.004 rpy=-1.57 0 0
- added joint fc1/imu_joint: type fixed, parent fc1/base_link, child fc1/imu_link, origin xyz=0.0 0 0.068 rpy=0 0 0
- added joint fc1/scan_joint: type fixed, parent fc1/base_link, child fc1/base_scan, origin xyz=-0.064 0 0.122 rpy=0 0 0
- added joint fc1/wheel_left_joint: type continuous, parent fc1/base_link, child fc1/wheel_left_link, origin xyz=0.0 0.144 0.023 rpy=-1.57 0 0, axis 0 0 1
- added joint fc1/wheel_right_joint: type continuous, parent fc1/base_link, child fc1/wheel_right_link, origin xyz=0.0 -0.144 0.023 rpy=-1.57 0 0, axis 0 0 1
