Commit message: multi robot localization

File: follow_cart/urdf/convoy/jetbot.gazebo.xacro (robot description, xacro)
@@ -20,26 +20,4 @@
     <maxVel>0.5</maxVel>
     <fdir1>1 0 0</fdir1>
-  </gazebo>
-  <gazebo>
-    <plugin name="diff_drive_controller" filename="libgazebo_ros_diff_drive.so">
-      <commandTopic>cmd_vel</commandTopic>
-      <odometryTopic>odom</odometryTopic>
-      <odometryFrame>odom</odometryFrame>
-      <odometrySource>encoder</odometrySource>
-      <publishOdomTF>true</publishOdomTF>
-      <robotBaseFrame>base_footprint</robotBaseFrame>
-      <publishWheelTF>false</publishWheelTF>
-      <publishTf>true</publishTf>
-      <publishWheelJointState>true</publishWheelJointState>
-      <legacyMode>false</legacyMode>
-      <updateRate>30</updateRate>
-      <leftJoint>left_wheel_hinge</leftJoint>
-      <rightJoint>right_wheel_hinge</rightJoint>
-      <wheelSeparation>0.096</wheelSeparation>
-      <wheelDiameter>0.065</wheelDiameter>
-      <wheelAcceleration>1</wheelAcceleration>
-      <wheelTorque>1</wheelTorque>
-      <rosDebugLevel>na</rosDebugLevel>
-    </plugin>
   </gazebo>
   <gazebo reference="camera_link">

File: follow_cart/urdf/follow_cart/turtlebot3_waffle_pi.urdf (robot description, URDF)
Before this commit: robot turtlebot3_waffle_pi, 8 links, 7 joints
Links:
- removed link fc1/base_footprint
- removed link fc1/base_link
- removed link fc1/base_scan
- removed link fc1/caster_back_left_link
- removed link fc1/caster_back_right_link
- removed link fc1/imu_link
- removed link fc1/wheel_left_link
- removed link fc1/wheel_right_link
- added link base_footprint
- added link base_link, mass 1.3729096e+00; collision box size=0.266 0.266 0.094; visual mesh filename=file://$(find turtlebot3_description)/meshes/bases/waffle_p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 scale=0.001 0.001 0.001
- added link base_scan, mass 0.114; collision cylinder length=0.0315 radius=0.055; visual mesh filename=file://$(find turtlebot3_description)/meshes/sensors/lds.stl scale=0.001 0.001 0.001
- added link caster_back_left_link, mass 0.005; collision box size=0.030 0.009 0.020
- added link caster_back_right_link, mass 0.005; collision box size=0.030 0.009 0.020
- added link imu_link
- added link wheel_left_link, mass 2.8498940e-02; collision cylinder length=0.018 radius=0.033; visual mesh filename=file://$(find turtlebot3_description)/meshes/wheels/left_ti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 scale=0.001 0.001 0.001
- added link wheel_right_link, mass 2.8498940e-02; collision cylinder length=0.018 radius=0.033; visual mesh filename=file://$(find turtlebot3_description)/meshes/wheels/right_t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 scale=0.001 0.001 0.001
Joints:
- removed joint fc1/base_joint
- removed joint fc1/caster_back_left_joint
- removed joint fc1/caster_back_right_joint
- removed joint fc1/imu_joint
- removed joint fc1/scan_joint
- removed joint fc1/wheel_left_joint
- removed joint fc1/wheel_right_joint
- added joint base_joint: type fixed, parent base_footprint, child base_link, origin xyz=0 0 0.010 rpy=0 0 0
- added joint caster_back_left_joint: type fixed, parent base_link, child caster_back_left_link, origin xyz=-0.177 0.064 -0.004 rpy=-1.57 0 0
- added joint caster_back_right_joint: type fixed, parent base_link, child caster_back_right_link, origin xyz=-0.177 -0.064 -0.004 rpy=-1.57 0 0
- added joint imu_joint: type fixed, parent base_link, child imu_link, origin xyz=0.0 0 0.068 rpy=0 0 0
- added joint scan_joint: type fixed, parent base_link, child base_scan, origin xyz=-0.064 0 0.122 rpy=0 0 0
- added joint wheel_left_joint: type continuous, parent base_link, child wheel_left_link, origin xyz=0.0 0.144 0.023 rpy=-1.57 0 0, axis 0 0 1
- added joint wheel_right_joint: type continuous, parent base_link, child wheel_right_link, origin xyz=0.0 -0.144 0.023 rpy=-1.57 0 0, axis 0 0 1

Commit message: tf odom->base_footprint 해결

File: follow_cart/urdf/convoy/jetbot.gazebo.xacro (robot description, xacro)
@@ -1,7 +1,5 @@
 <?xml version="1.0" ?>
 <robot name="JetBot_sim"  xmlns:xacro="http://ros.org/wiki/xacro">
-  <xacro:arg name="camera_visualize" default="true"/>
-  <xacro:arg name="laser_visualize"  default="false"/>
-  <gazebo reference="left_wheel">
+  <gazebo reference="convoy/wheel_left_link">
     <mu1>0.1</mu1>
     <mu2>0.1</mu2>
@@ -12,5 +10,5 @@
     <fdir1>1 0 0</fdir1>
   </gazebo>
-  <gazebo reference="right_wheel">
+  <gazebo reference="convoy/wheel_right_link">
     <mu1>0.1</mu1>
     <mu2>0.1</mu2>
@@ -21,71 +19,204 @@
     <fdir1>1 0 0</fdir1>
   </gazebo>
-  <gazebo reference="camera_link">
-    <sensor type="camera" name="camera">
-      <always_on>true</always_on>
-      <visualize>$(arg camera_visualize)</visualize>
-      <camera>
+  <gazebo reference="convoy/camera_link">
+    <sensor name='camera' type='camera'>
+        <always_on>1</always_on>
+        <visualize>1</visualize>
+        <camera>
           <horizontal_fov>2.79253</horizontal_fov>
           <image>
-              <width>1280</width>
-              <height>720</height>
-              <format>R8G8B8</format>
+            <width>1280</width>
+            <height>720</height>
+            <format>R8G8B8</format>
           </image>
           <clip>
-              <near>0.01</near>
-              <far>1</far>
+            <near>0.01</near>
+            <far>1</far>
           </clip>
           <noise>
             <type>gaussian</type>
-            <mean>0.0</mean>
+            <mean>0</mean>
             <stddev>0.01</stddev>
           </noise>
-      </camera>
-      <plugin name="camera_controller" filename="libgazebo_ros_camera.so">
-        <alwaysOn>true</alwaysOn>
-        <updateRate>30.0</updateRate>
-        <cameraName>camera</cameraName>
-        <frameName>camera_link</frameName>
-        <imageTopicName>rgb/image_raw</imageTopicName>
-        <cameraInfoTopicName>rgb/camera_info</cameraInfoTopicName>
-        <hackBaseline>0.07</hackBaseline>
-        <distortionK1>0.0</distortionK1>
-        <distortionK2>0.0</distortionK2>
-        <distortionK3>0.0</distortionK3>
-        <distortionT1>0.0</distortionT1>
-        <distortionT2>0.0</distortionT2>
-      </plugin>
+        </camera>
+        <plugin name='camera_controller' filename='libgazebo_ros_camera.so'>
+          <ros>
+            <namespace>/convoy</namespace>
+            <remapping>~/out:=image_raw</remapping>
+          </ros>
+          <alwaysOn>1</alwaysOn>
+          <updateRate>30.0</updateRate>
+          <cameraName>camera</cameraName>
+          <frameName>convoy/camera_link</frameName>
+          <imageTopicName>rgb/image_raw</imageTopicName>
+          <cameraInfoTopicName>rgb/camera_info</cameraInfoTopicName>
+          <hackBaseline>0.07</hackBaseline>
+          <distortionK1>0.0</distortionK1>
+          <distortionK2>0.0</distortionK2>
+          <distortionK3>0.0</distortionK3>
+          <distortionT1>0.0</distortionT1>
+          <distortionT2>0.0</distortionT2>
+        </plugin>
+        <pose>0.065 0 0.0957 0 0.25 0</pose>
+      </sensor>
+  </gazebo>
+  <gazebo reference="convoy/base_scan">
+      <sensor name='lds_lfcd_sensor' type='ray'>
+        <always_on>1</always_on>
+        <visualize>0</visualize>
+        <update_rate>5</update_rate>
+        <ray>
+          <scan>
+            <horizontal>
+              <samples>428</samples>
+              <resolution>0.84</resolution>
+              <min_angle>0</min_angle>
+              <max_angle>6.28319</max_angle>
+            </horizontal>
+          </scan>
+          <range>
+            <min>0.1</min>
+            <max>8</max>
+            <resolution>0.01</resolution>
+          </range>
+          <noise>
+            <type>gaussian</type>
+            <mean>0</mean>
+            <stddev>0.01</stddev>
+          </noise>
+        </ray>
+        <plugin name='scan' filename='libgazebo_ros_ray_sensor.so'>
+          <ros>
+            <namespace>/convoy</namespace>
+            <remapping>~/out:=scan</remapping>
+          </ros>
+          <output_type>sensor_msgs/LaserScan</output_type>
+          <frameName>convoy/base_scan</frameName>
+        </plugin>
+        <pose>0 -0.0058 0.137 0 -0 3.14</pose>
     </sensor>
   </gazebo>
-  <gazebo reference="lidar_link">
-    <sensor type="ray" name="lds_lfcd_sensor">
-      <pose>0 0 0 0 0 0</pose>
-      <visualize>$(arg laser_visualize)</visualize>
-      <update_rate>5</update_rate>
-      <ray>
-        <scan>
-          <horizontal>
-            <samples>428</samples>
-            <resolution>0.84</resolution>
-            <min_angle>0</min_angle>
-            <max_angle>6.28319</max_angle>
-          </horizontal>
-        </scan>
-        <range>
-          <min>0.1</min>
-          <max>8</max>
-          <resolution>0.01</resolution>
-        </range>
-        <noise>
-          <type>gaussian</type>
-          <mean>0.0</mean>
-          <stddev>0.01</stddev>
-        </noise>
-      </ray>
-      <plugin name="gazebo_ros_lds_lfcd_controller" filename="libgazebo_ros_laser.so">
-        <topicName>scan</topicName>
-        <frameName>lidar_link</frameName>
-      </plugin>
+  <gazebo reference="convoy/imu_link">
+    <sensor name="imu" type="imu">
+          <always_on>true</always_on>
+          <update_rate>100</update_rate>
+          <visualize>true</visualize>
+          <imu>
+            <orientation>
+              <x>
+                <noise type="gaussian">
+                  <mean>0.0</mean>
+                  <stddev>2e-3</stddev>
+                </noise>
+              </x>
+              <y>
+                <noise type="gaussian">
+                  <mean>0.0</mean>
+                  <stddev>2e-3</stddev>
+                </noise>
+              </y>
+              <z>
+                <noise type="gaussian">
+                  <mean>0.0</mean>
+                  <stddev>2e-3</stddev>
+                </noise>
+              </z>
+            </orientation>
+            <angular_velocity>
+              <x>
+                <noise type="gaussian">
+                  <mean>0.0</mean>
+                  <stddev>2e-4</stddev>
+                </noise>
+              </x>
+              <y>
+                <noise type="gaussian">
+                  <mean>0.0</mean>
+                  <stddev>2e-4</stddev>
+                </noise>
+              </y>
+              <z>
+                <noise type="gaussian">
+                  <mean>0.0</mean>
+                  <stddev>2e-4</stddev>
+                </noise>
+              </z>
+            </angular_velocity>
+            <linear_acceleration>
+              <x>
+                <noise type="gaussian">
+                  <mean>0.0</mean>
+                  <stddev>1.7e-2</stddev>
+                </noise>
+              </x>
+              <y>
+                <noise type="gaussian">
+                  <mean>0.0</mean>
+                  <stddev>1.7e-2</stddev>
+                </noise>
+              </y>
+              <z>
+                <noise type="gaussian">
+                  <mean>0.0</mean>
+                  <stddev>1.7e-2</stddev>
+                </noise>
+              </z>
+            </linear_acceleration>
+          </imu>
+          <plugin name="imu" filename="libgazebo_ros_imu_sensor.so">
+            <ros>
+              <namespace>/convoy</namespace>
+              <remapping>~/out:=imu</remapping>
+            </ros>
+            <initial_orientation_as_reference>false</initial_orientation_as_reference>
+            <frame_name>convoy/imu_link</frame_name>
+          </plugin>
     </sensor>
   </gazebo>
+  <gazebo>
+    <plugin name='scan' filename='libgazebo_ros_ray_sensor.so'>
+          <ros>
+            <namespace>/convoy</namespace>
+            <remapping>~/out:=scan</remapping>
+          </ros>
+          <output_type>sensor_msgs/LaserScan</output_type>
+          <frameName>convoy/base_scan</frameName>
+    </plugin>
+    <plugin name="imu" filename="libgazebo_ros_imu_sensor.so">
+            <ros>
+              <namespace>/convoy</namespace>
+              <remapping>~/out:=imu</remapping>
+            </ros>
+            <frame_name>convoy/imu_link</frame_name>
+    </plugin>
+    <plugin name='diff_drive' filename='libgazebo_ros_diff_drive.so'>
+      <ros>
+        <namespace>/convoy</namespace>
+      </ros>
+      <update_rate>30</update_rate>
+      <left_joint>convoy/wheel_left_joint</left_joint>
+      <right_joint>convoy/wheel_right_joint</right_joint>
+      <wheel_separation>0.096</wheel_separation>
+      <wheel_diameter>0.065</wheel_diameter>
+      <command_topic>cmd_vel</command_topic>
+      <odometry_topic>odom</odometry_topic>
+      <max_wheel_acceleration>1</max_wheel_acceleration>
+      <max_wheel_torque>1</max_wheel_torque>
+      <publish_odom>true</publish_odom>
+      <publish_odom_tf>true</publish_odom_tf>
+      <publish_wheel_tf>true</publish_wheel_tf>
+      <odometry_frame>convoy/odom</odometry_frame>
+      <robot_base_frame>convoy/base_footprint</robot_base_frame>
+      <odometry_source>1</odometry_source>
+    </plugin>
+    <plugin name="joint_state" filename="libgazebo_ros_joint_state_publisher.so">
+        <ros>
+          <namespace>/convoy</namespace>
+          <remapping>~/out:=joint_states</remapping>
+        </ros>
+        <update_rate>30</update_rate>
+        <joint_name>convoy/wheel_left_joint</joint_name>
+        <joint_name>convoy/wheel_right_joint</joint_name>
+    </plugin>
+  </gazebo>
 </robot>

File: follow_cart/urdf/convoy/jetbot.urdf (robot description, URDF)
Before this commit: robot JetBot, 7 links, 6 joints
Links:
- removed link base_footprint
- removed link base_link
- removed link base_scan
- removed link camera_link
- removed link imu_link
- removed link wheel_left_link
- removed link wheel_right_link
- added link convoy/base_footprint
- added link convoy/base_link, mass 1.0; collision mesh filename=file://$(find follow_cart)/meshes/convoy/JetBot-v3-Chassis.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 scale=0.001 0.001 0.001; visual mesh filename=file://$(find follow_cart)/meshes/convoy/JetBot-v3-Chassis.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 scale=0.001 0.001 0.001
- added link convoy/base_scan, mass 0.0; collision mesh filename=file://$(find follow_cart)/meshes/convoy/lidar-base.dae scale=1.0 1.0 1.0; visual mesh filename=file://$(find follow_cart)/meshes/convoy/lidar-base.dae scale=1.0 1.0 1.0
- added link convoy/camera_link, mass 0.01; visual box size=0.001 0.001 0.001
- added link convoy/imu_link
- added link convoy/wheel_left_link, mass 0.1; collision cylinder length=0.008 radius=0.030; visual mesh filename=file://$(find follow_cart)/meshes/convoy/JetBot-v3-Wheel.stl scale=0.001 0.001 0.001
- added link convoy/wheel_right_link, mass 0.1; collision cylinder length=0.008 radius=0.030; visual mesh filename=file://$(find follow_cart)/meshes/convoy/JetBot-v3-Wheel.stl scale=0.001 0.001 0.001
Joints:
- removed joint base_joint
- removed joint camera_joint
- removed joint imu_joint
- removed joint lidar_joint
- removed joint wheel_left_joint
- removed joint wheel_right_joint
- added joint convoy/base_joint: type fixed, parent convoy/base_footprint, child convoy/base_link, origin xyz=0.0 0.0 0.010 rpy=0 0 0
- added joint convoy/camera_joint: type fixed, parent convoy/base_link, child convoy/camera_link, origin xyz=0.065   0      0.0857 rpy=0    0.25  0, axis 0.96891  0       0.2474
- added joint convoy/imu_joint: type fixed, parent convoy/base_link, child convoy/imu_link, origin xyz=0 0 0.01
- added joint convoy/lidar_joint: type fixed, parent convoy/base_link, child convoy/base_scan, origin xyz=0.0 -0.0058  0.127 rpy=0   0   3.14, axis 0 0 0
- added joint convoy/wheel_left_joint: type continuous, parent convoy/base_link, child convoy/wheel_left_link, origin xyz=0.03     0.05125  0.03 rpy=0       0       1.57079, axis 1  0  0
- added joint convoy/wheel_right_joint: type continuous, parent convoy/base_link, child convoy/wheel_right_link, origin xyz=0.03   -0.0595  0.03 rpy=0       0       1.57079, axis 1  0  0

File: follow_cart/urdf/follow_cart/turtlebot3_waffle_pi.urdf (robot description, URDF)
Before this commit: robot turtlebot3_waffle_pi, 8 links, 7 joints
Links:
- removed link base_footprint
- removed link base_link
- removed link base_scan
- removed link caster_back_left_link
- removed link caster_back_right_link
- removed link imu_link
- removed link wheel_left_link
- removed link wheel_right_link
- added link $(arg robot_name)/base_footprint
- added link $(arg robot_name)/base_link, mass 1.3729096e+00; collision box size=0.266 0.266 0.094; visual mesh filename=file://$(find turtlebot3_description)/meshes/bases/waffle_p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 scale=0.001 0.001 0.001
- added link $(arg robot_name)/base_scan, mass 0.114; collision cylinder length=0.0315 radius=0.055; visual mesh filename=file://$(find turtlebot3_description)/meshes/sensors/lds.stl scale=0.001 0.001 0.001
- added link $(arg robot_name)/caster_back_left_link, mass 0.005; collision box size=0.030 0.009 0.020
- added link $(arg robot_name)/caster_back_right_link, mass 0.005; collision box size=0.030 0.009 0.020
- added link $(arg robot_name)/imu_link
- added link $(arg robot_name)/wheel_left_link, mass 2.8498940e-02; collision cylinder length=0.018 radius=0.033; visual mesh filename=file://$(find turtlebot3_description)/meshes/wheels/left_ti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 scale=0.001 0.001 0.001
- added link $(arg robot_name)/wheel_right_link, mass 2.8498940e-02; collision cylinder length=0.018 radius=0.033; visual mesh filename=file://$(find turtlebot3_description)/meshes/wheels/right_t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 scale=0.001 0.001 0.001
Joints:
- removed joint base_joint
- removed joint caster_back_left_joint
- removed joint caster_back_right_joint
- removed joint imu_joint
- removed joint scan_joint
- removed joint wheel_left_joint
- removed joint wheel_right_joint
- added joint $(arg robot_name)/base_joint: type fixed, parent $(arg robot_name)/base_footprint, child $(arg robot_name)/base_link, origin xyz=0 0 0.010 rpy=0 0 0
- added joint $(arg robot_name)/caster_back_left_joint: type fixed, parent $(arg robot_name)/base_link, child $(arg robot_name)/caster_back_left_link, origin xyz=-0.177 0.064 -0.004 rpy=-1.57 0 0
- added joint $(arg robot_name)/caster_back_right_joint: type fixed, parent $(arg robot_name)/base_link, child $(arg robot_name)/caster_back_right_link, origin xyz=-0.177 -0.064 -0.004 rpy=-1.57 0 0
- added joint $(arg robot_name)/imu_joint: type fixed, parent $(arg robot_name)/base_link, child $(arg robot_name)/imu_link, origin xyz=0.0 0 0.068 rpy=0 0 0
- added joint $(arg robot_name)/scan_joint: type fixed, parent $(arg robot_name)/base_link, child $(arg robot_name)/base_scan, origin xyz=-0.064 0 0.122 rpy=0 0 0
- added joint $(arg robot_name)/wheel_left_joint: type continuous, parent $(arg robot_name)/base_link, child $(arg robot_name)/wheel_left_link, origin xyz=0.0 0.144 0.023 rpy=-1.57 0 0, axis 0 0 1
- added joint $(arg robot_name)/wheel_right_joint: type continuous, parent $(arg robot_name)/base_link, child $(arg robot_name)/wheel_right_link, origin xyz=0.0 -0.144 0.023 rpy=-1.57 0 0, axis 0 0 1
