Commit message: 후미 차량 카메라 추가

File: follow_cart/urdf/convoy/turtlebot3_waffle_pi.urdf (robot description, URDF)
Before this commit: robot turtlebot3_waffle_pi, 11 links, 10 joints
Joints:
- joint $(arg robot_name)/camera_rgb_optical_joint: origin xyz=0 0 0 rpy=-1.57 0 -1.57 -> xyz=0 0 0 rpy=0 0 0

File: follow_cart/urdf/follow_cart/follow_cart_1.urdf (robot description, URDF)
Before this commit: robot turtlebot3_waffle_pi, 11 links, 10 joints
Joints:
- joint $(arg robot_name)/camera_joint: origin xyz=0.073 -0.161 0.084 rpy=0 0 -0.785 -> xyz=0.063 -0.14 0.084 rpy=0 0 -0.785
- joint $(arg robot_name)/camera_rgb_optical_joint: origin xyz=0 0 0 rpy=-1.57 0 -1.57 -> xyz=0 0 0 rpy=0 0 0

File: follow_cart/urdf/follow_cart/follow_cart_2.urdf (robot description, URDF)
Before this commit: robot turtlebot3_waffle_pi, 11 links, 10 joints
Joints:
- joint $(arg robot_name)/camera_rgb_optical_joint: origin xyz=0 0 0 rpy=-1.57 0 -1.57 -> xyz=0 0 0 rpy=0 0 0

File: follow_cart/urdf/follow_cart/follow_cart_3.urdf (robot description, URDF)
Before this commit: robot turtlebot3_waffle_pi, 11 links, 10 joints
Joints:
- joint $(arg robot_name)/camera_joint: origin xyz=0.073 0.161 0.084 rpy=0 0 0.785 -> xyz=0.063 0.14 0.084 rpy=0 0 0.785
- joint $(arg robot_name)/camera_rgb_optical_joint: origin xyz=0 0 0 rpy=-1.57 0 -1.57 -> xyz=0 0 0 rpy=0 0 0
