Commit message: 모델에서 카메라 발행을 못함

File: follow_cart/urdf/follow_cart/turtlebot3_waffle_pi.urdf (robot description, URDF)
Before this commit: robot turtlebot3_waffle_pi, 8 links, 7 joints
Links:
- removed link base_footprint
- removed link base_link
- removed link base_scan
- removed link caster_back_left_link
- removed link caster_back_right_link
- removed link imu_link
- removed link wheel_left_link
- removed link wheel_right_link
- added link $(arg robot_name)/base_footprint
- added link $(arg robot_name)/base_link, mass 1.3729096e+00; collision box size=0.266 0.266 0.094; visual mesh filename=file://$(find turtlebot3_description)/meshes/bases/waffle_p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 scale=0.001 0.001 0.001
- added link $(arg robot_name)/base_scan, mass 0.114; collision cylinder length=0.0315 radius=0.055; visual mesh filename=file://$(find turtlebot3_description)/meshes/sensors/lds.stl scale=0.001 0.001 0.001
- added link $(arg robot_name)/camera_link; collision box size=0.015 0.030 0.027
- added link $(arg robot_name)/camera_rgb_frame
- added link $(arg robot_name)/camera_rgb_optical_frame
- added link $(arg robot_name)/caster_back_left_link, mass 0.005; collision box size=0.030 0.009 0.020
- added link $(arg robot_name)/caster_back_right_link, mass 0.005; collision box size=0.030 0.009 0.020
- added link $(arg robot_name)/imu_link
- added link $(arg robot_name)/wheel_left_link, mass 2.8498940e-02; collision cylinder length=0.018 radius=0.033; visual mesh filename=file://$(find turtlebot3_description)/meshes/wheels/left_ti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 scale=0.001 0.001 0.001
- added link $(arg robot_name)/wheel_right_link, mass 2.8498940e-02; collision cylinder length=0.018 radius=0.033; visual mesh filename=file://$(find turtlebot3_description)/meshes/wheels/right_t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 scale=0.001 0.001 0.001
Joints:
- removed joint base_joint
- removed joint caster_back_left_joint
- removed joint caster_back_right_joint
- removed joint imu_joint
- removed joint scan_joint
- removed joint wheel_left_joint
- removed joint wheel_right_joint
- added joint $(arg robot_name)/base_joint: type fixed, parent $(arg robot_name)/base_footprint, child $(arg robot_name)/base_link, origin xyz=0 0 0.010 rpy=0 0 0
- added joint $(arg robot_name)/camera_joint: type fixed, parent $(arg robot_name)/base_link, child $(arg robot_name)/camera_link, origin xyz=0.073 -0.011 0.084 rpy=0 0 0
- added joint $(arg robot_name)/camera_rgb_joint: type fixed, parent $(arg robot_name)/camera_link, child $(arg robot_name)/camera_rgb_frame, origin xyz=0.003 0.011 0.009 rpy=0 0 0
- added joint $(arg robot_name)/camera_rgb_optical_joint: type fixed, parent $(arg robot_name)/camera_rgb_frame, child $(arg robot_name)/camera_rgb_optical_frame, origin xyz=0 0 0 rpy=-1.57 0 -1.57
- added joint $(arg robot_name)/caster_back_left_joint: type fixed, parent $(arg robot_name)/base_link, child $(arg robot_name)/caster_back_left_link, origin xyz=-0.177 0.064 -0.004 rpy=-1.57 0 0
- added joint $(arg robot_name)/caster_back_right_joint: type fixed, parent $(arg robot_name)/base_link, child $(arg robot_name)/caster_back_right_link, origin xyz=-0.177 -0.064 -0.004 rpy=-1.57 0 0
- added joint $(arg robot_name)/imu_joint: type fixed, parent $(arg robot_name)/base_link, child $(arg robot_name)/imu_link, origin xyz=0.0 0 0.068 rpy=0 0 0
- added joint $(arg robot_name)/scan_joint: type fixed, parent $(arg robot_name)/base_link, child $(arg robot_name)/base_scan, origin xyz=-0.064 0 0.122 rpy=0 0 0
- added joint $(arg robot_name)/wheel_left_joint: type continuous, parent $(arg robot_name)/base_link, child $(arg robot_name)/wheel_left_link, origin xyz=0.0 0.144 0.023 rpy=-1.57 0 0, axis 0 0 1
- added joint $(arg robot_name)/wheel_right_joint: type continuous, parent $(arg robot_name)/base_link, child $(arg robot_name)/wheel_right_link, origin xyz=0.0 -0.144 0.023 rpy=-1.57 0 0, axis 0 0 1
