Commit message: 카메라 사용 대형유지 로직 구성

File: follow_cart/urdf/follow_cart/follow_cart_1.urdf (robot description, URDF)
Before this commit: robot turtlebot3_waffle_pi, 11 links, 10 joints
Joints:
- joint $(arg robot_name)/camera_joint: origin xyz=0.063 -0.14 0.084 rpy=0 0 -0.785 -> xyz=0.073 -0.011 0.084 rpy=0 0.5 0

File: follow_cart/urdf/follow_cart/follow_cart_2.urdf (robot description, URDF)
Before this commit: robot turtlebot3_waffle_pi, 11 links, 10 joints
Joints:
- joint $(arg robot_name)/camera_joint: origin xyz=0.073 -0.011 0.084 rpy=0 0 0 -> xyz=0.063 -0.14 0.084 rpy=0 0 -0.785
